Commit message: Swap in re-exported Palpador/Wire Drum/User Step meshes + fix placement
Co-Authored-By: Claude Opus 4.8 <noreply@anthropic.com>

File: apps/dev-host/assets/M600_PRO/M600_PRO.urdf (robot description, URDF)
Before this commit: robot M600_PRO, 25 links, 24 joints
Links:
- link palpador_pro_link: geometry visual mesh filename=Palpador PRO.glb scale=1 1 1
- link user_step_link: geometry visual mesh filename=User Step.glb scale=1 1 1
- link wire_drum_link: geometry visual mesh filename=Wire Drum.glb scale=1 1 1

Commit message: M600: swap in the 2026-09 re-exported assemblies
Replace 22 URDF meshes (18 files) with the new CAD re-exports and add the
HRS050-AF-20 chiller, which the viewer loads but the repo never shipped.

The exports are in metres with their axes re-oriented per file, so each URDF
visual got scale 1 and a new rpy/xyz solved by vertex-to-surface fit against
the previous mesh in its link frame (mean error 0.2-7.8 mm, ICP off-axis drift
<0.25 deg). Wire Drum keeps its old rotation (same frame, units only).

Materials were stripped by the exporter, so every material-less primitive gets
one brushed-steel texture (box-projected UVs, 0.25 m tile, mirrored repeat).
The front door's window pane is re-baked as transmissive glass.

Chassis (empty export) and Wire Drum Door (wrong-sized export) are unchanged.

Co-Authored-By: Claude Opus 5.5 <noreply@anthropic.com>

File: apps/dev-host/assets/M600_PRO/M600_PRO.urdf (robot description, URDF)
Before this commit: robot M600_PRO, 25 links, 24 joints
Links:
- link central_feeder_wheel_link: geometry visual mesh filename=Central Feeder Wheel.glb scale=1 1 1
- link display_link: geometry visual mesh filename=Display.glb scale=1 1 1
- link eje_x_link: geometry visual mesh filename=Eje X.glb scale=1 1 1
- link eje_y_link: geometry visual mesh filename=Eje Y.glb scale=1 1 1
- link feeder_link: geometry visual mesh filename=Feeder.glb scale=1 1 1
- link front_door_link: geometry visual mesh filename=Front Door.glb scale=1 1 1
- link gas_spring_main_part_left_link: geometry visual mesh filename=Gas Spring Main Part Left.glb scale=1 1 1
- link gas_spring_main_part_right_link: geometry visual mesh filename=Gas Spring Main Part Right.glb scale=1 1 1
- link gas_spring_secondary_part_left_link: geometry visual mesh filename=Gas Spring Secondary Part Left.glb scale=1 1 1
- link gas_spring_secondary_part_right_link: geometry visual mesh filename=Gas Spring Secondary Part Right.glb scale=1 1 1
- link handle_link: geometry visual mesh filename=Handle.glb scale=1 1 1
- link head_link: geometry visual mesh filename=Head.glb scale=1 1 1
- link left_feeder_wheel_link: geometry visual mesh filename=Left Feeder Wheel.glb scale=1 1 1
- link palpador_pro_link: geometry visual mesh filename=Palpador PRO.glb scale=1 1 1
- link right_feeder_wheel_link: geometry visual mesh filename=Right Feeder Wheel.glb scale=1 1 1
- link spool_1_link: geometry visual mesh filename=Spool Cooper.glb scale=1 1 1
- link spool_2_link: geometry visual mesh filename=Spool Stainless Steel.glb scale=1 1 1
- link spools_door_link: geometry visual mesh filename=Spools Door.glb scale=1 1 1
- link top_cover_link: geometry visual mesh filename=Top Cover.glb scale=1 1 1
- link user_step_link: geometry visual mesh filename=User Step.glb scale=1 1 1
- link wire_drum_link: geometry visual mesh filename=Wire Drum.glb scale=1 1 1
- link z_axis_link: geometry visual mesh filename=Z axis.glb scale=1 1 1

Commit message: M600: give the re-exported parts the original June look; real Wire Drum Door
The 2026-09-25 CAD exports carry no materials. Each triangle of the new
meshes now takes the material of the nearest surface of the original June
mesh (same link frame, 5-sample vote), so panels, trim, buttons, spools and
the chiller read as before. Textures (logos, screen image) do not carry over.
The door glass and nozzle tag are kept.

Wire Drum Door: the export also contains a stray copy of the Top Cover; the
door object alone (31x197x265 mm, same as before) is fitted onto the old
door (1.2 mm mean) and replaces it.

Co-Authored-By: Claude Opus 5.5 <noreply@anthropic.com>

File: apps/dev-host/assets/M600_PRO/M600_PRO.urdf (robot description, URDF)
Before this commit: robot M600_PRO, 25 links, 24 joints
Links:
- link wire_spool_door_link: geometry visual mesh filename=Wire Drum Door.glb scale=1 1 1

Commit message: M600: texture-atlas test on Spools Door + Wire Drum Door (2026-09-29 export)
Bind the first baked PBR atlas to the two door assemblies. The delivered
GLBs name their materials Test_Metal_Atlas / Test_Plastic_Atlas but embed no
images, so new Spools Door_atlas.glb / Wire Drum Door_atlas.glb reference the
PNGs in assets/M600_PRO/Textures/ (Metallic + Roughness packed into one glTF
metallicRoughness map, factors reset to 1). URDF repointed; the previous door
files stay for rollback. Geometry placement is unchanged.

tuneMaterial leaves materials named *_Atlas at metalness/roughness 1 (the
flat 0.24/0.66 overrides would multiply the maps) and gives them the scoped
studio env map, as the feeder wheels already get. Detection is by name only.
Atlas PNGs under apps/dev-host/assets are LFS-tracked.

Kept 4096 px and the plastic atlas as delivered per Maksim; its Metallic map
matches the metal one and is flagged for re-bake.

Co-Authored-By: Claude Fable 5.1 <noreply@anthropic.com>

File: apps/dev-host/assets/M600_PRO/M600_PRO.urdf (robot description, URDF)
Before this commit: robot M600_PRO, 25 links, 24 joints
Links:
- link spools_door_link: geometry visual mesh filename=Spools Door_atlas.glb scale=1 1 1
- link wire_spool_door_link: geometry visual mesh filename=Wire Drum Door_atlas.glb scale=1 1 1

Commit message: Viewer: 2026-10-22 textured re-exports — 10 M600 parts on the PBR atlases
Port of the local design-system-v3 commits 9e967c7f, 543e6465, 51fd21aa.

Maksim's second atlas delivery (D:/UI_UX/M600 Pro_glb/glb_2_test_atlas, Blender
3.6): Display, Front Door, Gas Spring Main/Secondary, Handle, Spools Door,
Top Cover, Wire Drum Door, Wire Drum, plus Locking Mechanism Base (built, not
placed — no link in the assembly yet).

- New <Part>_2210.glb files reference the loose PNGs in Textures/ (2K working
  copies, 4K originals in Textures/4k/). Metal atlas unchanged; plastic atlas
  is a new bake (metallic ~0 now, was ~75 %) -> ?v=2k2; new Test_Metal_Atlas_2
  set for the "Test_Metal_Atlas_02" slot (hinge pins); Test_Display screen
  image bound as a plain baseColor map.
- Front door "Glass" slot rewritten to the Chamber Window Glass transmission
  recipe so tuneMaterial turns it into the 0.18-opacity pane (the door had been
  one opaque solid since the Sep-28 swap).
- Gas spring Left/Right links share one file. Visual origins unchanged: every
  link verified to land where the current mesh is (live __links() diff against
  the previous assembly: 0 mm on all 25 links; the current meshes here are
  byte-identical to the local ones the check ran against).
- ATLAS_MATERIAL_NAME_RE accepts numbered variants (_atlas_02).
- apps/dev-host/tools/build_atlas_glbs.py: the binding/packing/placement tool,
  kept in the repo (the Oct-13 scratchpad version was lost).

Gate: bash gate.sh 9/9 green.

Co-Authored-By: Claude Fable 5.1 <noreply@anthropic.com>

File: apps/dev-host/assets/M600_PRO/M600_PRO.urdf (robot description, URDF)
Before this commit: robot M600_PRO, 25 links, 24 joints
Links:
- link display_link: geometry visual mesh filename=Display_2210.glb scale=1 1 1
- link front_door_link: geometry visual mesh filename=Front Door_2210.glb scale=1 1 1
- link gas_spring_main_part_left_link: geometry visual mesh filename=Gas Spring Main Part_2210.glb scale=1 1 1
- link gas_spring_main_part_right_link: geometry visual mesh filename=Gas Spring Main Part_2210.glb scale=1 1 1
- link gas_spring_secondary_part_left_link: geometry visual mesh filename=Gas Spring Secondary Part_2210.glb scale=1 1 1
- link gas_spring_secondary_part_right_link: geometry visual mesh filename=Gas Spring Secondary Part_2210.glb scale=1 1 1
- link handle_link: geometry visual mesh filename=Handle_2210.glb scale=1 1 1
- link spools_door_link: geometry visual mesh filename=Spools Door_2210.glb scale=1 1 1
- link top_cover_link: geometry visual mesh filename=Top Cover_2210.glb scale=1 1 1
- link wire_drum_link: geometry visual mesh filename=Wire Drum_2210.glb scale=1 1 1
- link wire_spool_door_link: geometry visual mesh filename=Wire Drum Door_2210.glb scale=1 1 1
